File: PCBs/MOL/MOL-v2-1.brd (EAGLE design)
At the start: 141 x 53.3 mm, 27 parts, among them IC1 ULN2803, IC2 ULN2803, J1 SERVO1, J10 JOY1, J11 JOY2, J2 SERVO2, J3 STRIPS, J4 ACTUATORS, J5 POWER-5V, J6 AN-IN-1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

Commit message: daniel tings
Connections:
- net B1 renamed BTN1
- net B10 renamed BTN10
- net B11 renamed BTN11
- net B12 renamed BTN12
- net B13 renamed BTN13
- net B14 renamed BTN14
- net B15 renamed BTN15
- net B16 renamed BTN16
- net B2 renamed BTN2
- net B3 renamed BTN3
- net B4 renamed BTN4
- net B5 renamed BTN5
- net B6 renamed BTN6
- net B7 renamed BTN7
- net B8 renamed BTN8
- net B9 renamed BTN9
- net JOY_AN_H_S renamed JOYH1
- net JOY_AN_V_M renamed JOYV2
- net JOY_AN_V_S renamed JOYV1
- net JOY_BTN_M renamed JOYB2
- net JOY_BTN_S renamed JOYB1
- removed net JOY_AN_H_M: J11.3
- net JOYH2: now also J11.3
Changed lines of the file:
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@@
 <via x="97.31375" y="17.78" extent="1-16" drill="0.381"/>
 </signal>
-<signal name="B1">
+<signal name="BTN1">
 <contactref element="J3" pad="3"/>
 <contactref element="TEENSY" pad="54"/>
@@
 <via x="71.12" y="16.1925" extent="1-16" drill="0.381"/>
 </signal>
-<signal name="B2">
+<signal name="BTN2">
 <contactref element="J3" pad="4"/>
 <contactref element="TEENSY" pad="56"/>
@@
 <via x="26.035" y="33.3375" extent="1-16" drill="0.381"/>
 </signal>
-<signal name="B3">
+<signal name="BTN3">
 <contactref element="J3" pad="13"/>
 <contactref element="TEENSY" pad="12"/>
@@
 <via x="26.9875" y="37.465" extent="1-16" drill="0.381"/>
 </signal>
-<signal name="B4">
+<signal name="BTN4">
 <contactref element="J3" pad="14"/>
 <contactref element="TEENSY" pad="24"/>
@@
 <via x="37.1475" y="39.6875" extent="1-16" drill="0.381"/>
 </signal>
-<signal name="B5">
+<signal name="BTN5">
 <contactref element="J3" pad="23"/>
 <contactref element="TEENSY" pad="1"/>
@@
 <wire x1="41.75125" y1="35.56" x2="41.656" y2="35.56" width="0.254" layer="16"/>
 </signal>
-<signal name="B7">
+<signal name="BTN7">
 <contactref element="J3" pad="33"/>
 <contactref element="TEENSY" pad="26"/>
@@
 </signal>
 <signal name="JOYH2" class="3">
+<contactref element="J11" pad="3"/>
 <contactref element="TEENSY" pad="31"/>
 <wire x1="92.3925" y1="32.385" x2="92.3925" y2="35.56" width="0.381" layer="16"/>
@@
 <wire x1="138.27125" y1="25.4" x2="131.7625" y2="31.90875" width="0.381" layer="1"/>
 <wire x1="92.3925" y1="35.56" x2="92.456" y2="35.56" width="0.381" layer="16"/>
+<wire x1="138.27125" y1="25.4" x2="138.303" y2="25.4" width="0.381" layer="1"/>
 <via x="92.3925" y="32.385" extent="1-16" drill="0.381"/>
 </signal>
-<signal name="JOY_AN_V_M" class="3">
+<signal name="JOYV2" class="3">
 <contactref element="J11" pad="4"/>
 <contactref element="TEENSY" pad="32"/>
@@
 <via x="95.40875" y="31.59125" extent="1-16" drill="0.381"/>
 </signal>
-<signal name="B12">
+<signal name="BTN12">
 <contactref element="J3" pad="54"/>
 <contactref element="TEENSY" pad="48"/>
@@
 <via x="87.15375" y="40.64" extent="1-16" drill="0.381"/>
 </signal>
-<signal name="B11">
+<signal name="BTN11">
 <contactref element="J3" pad="53"/>
 <contactref element="TEENSY" pad="52"/>
@@
 <via x="91.1225" y="37.30625" extent="1-16" drill="0.381"/>
 </signal>
-<signal name="B10">
+<signal name="BTN10">
 <contactref element="J3" pad="42"/>
 <contactref element="TEENSY" pad="40"/>
@@
 <via x="72.7075" y="28.2575" extent="1-16" drill="0.381"/>
 </signal>
-<signal name="B9">
+<signal name="BTN9">
 <contactref element="J3" pad="45"/>
 <contactref element="TEENSY" pad="27"/>
@@
 <via x="77.62875" y="50.00625" extent="1-16" drill="0.381"/>
 </signal>
-<signal name="B8">
+<signal name="BTN8">
 <contactref element="J3" pad="34"/>
 <contactref element="TEENSY" pad="25"/>
@@
 <wire x1="110.49" y1="29.21" x2="110.49" y2="25.4" width="0.254" layer="1"/>
 </signal>
-<signal name="B13">
+<signal name="BTN13">
 <contactref element="S5" pad="1"/>
 <contactref element="TEENSY" pad="42"/>
@@
 <via x="50.64125" y="2.2225" extent="1-16" drill="0.381"/>
 </signal>
-<signal name="B14">
+<signal name="BTN14">
 <contactref element="S6" pad="1"/>
 <contactref element="TEENSY" pad="51"/>
@@
 <wire x1="79.85125" y1="25.4" x2="79.756" y2="25.4" width="0.254" layer="16"/>
 </signal>
-<signal name="B15">
+<signal name="BTN15">
 <contactref element="S7" pad="1"/>
 <contactref element="TEENSY" pad="28"/>
@@
 <via x="83.185" y="6.6675" extent="1-16" drill="0.381"/>
 </signal>
-<signal name="JOY_AN_V_S" class="3">
+<signal name="JOYV1" class="3">
 <contactref element="J10" pad="4"/>
 <contactref element="TEENSY" pad="A10"/>
@@
 <via x="46.0375" y="26.19375" extent="1-16" drill="0.381"/>
 </signal>
-<signal name="JOY_AN_H_S" class="3">
+<signal name="JOYH1" class="3">
 <contactref element="J10" pad="3"/>
 <contactref element="TEENSY" pad="A11"/>
@@
 <wire x1="2.69875" y1="25.4" x2="2.667" y2="25.4" width="0.381" layer="1"/>
 </signal>
-<signal name="JOY_BTN_S">
+<signal name="JOYB1">
 <contactref element="J10" pad="5"/>
 <contactref element="TEENSY" pad="47"/>
@@
 <via x="2.38125" y="18.7325" extent="1-16" drill="0.381"/>
 </signal>
-<signal name="JOY_BTN_M">
+<signal name="JOYB2">
 <contactref element="J11" pad="5"/>
 <contactref element="TEENSY" pad="44"/>
@@
 <wire x1="120.65" y1="2.54" x2="124.7775" y2="6.6675" width="0.254" layer="16"/>
 </signal>
-<signal name="B16">
+<signal name="BTN16">
 <contactref element="S8" pad="1"/>
 <contactref element="TEENSY" pad="13"/>
@@
 <wire x1="136.04875" y1="9.8425" x2="136.144" y2="9.779" width="0.254" layer="16"/>
 </signal>
-<signal name="B6">
+<signal name="BTN6">
 <contactref element="TEENSY" pad="11"/>
 </signal>
@@
 <wire x1="89.916" y1="27.94" x2="90.01125" y2="27.94" width="0" layer="19" extent="16-16"/>
 </signal>
-<signal name="JOY_AN_H_M" class="3">
-<contactref element="J11" pad="3"/>
-</signal>
 </signals>
