File: PCBs/MOL/MOL-v2-1.sch (EAGLE design)
At the start: 29 parts, among them IC1 ULN2803, IC2 ULN2803, J1 SERVO1, J10 JOY1, J11 JOY2, J2 SERVO2, J3 STRIPS, J4 ACTUATORS, J5 POWER-5V, J6 AN-IN-1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

Commit message: daniel tings
Connections:
- net B1 renamed BTN1
- net B10 renamed BTN10
- net B11 renamed BTN11
- net B12 renamed BTN12
- net B13 renamed BTN13
- net B14 renamed BTN14
- net B15 renamed BTN15
- net B16 renamed BTN16
- net B2 renamed BTN2
- net B3 renamed BTN3
- net B4 renamed BTN4
- net B5 renamed BTN5
- net B6 renamed BTN6
- net B7 renamed BTN7
- net B8 renamed BTN8
- net B9 renamed BTN9
- net JOY_AN_H_S renamed JOYH1
- net JOY_AN_V_M renamed JOYV2
- net JOY_AN_V_S renamed JOYV1
- net JOY_BTN_M renamed JOYB2
- net JOY_BTN_S renamed JOYB1
- removed net JOY_AN_H_M: J11.3, MIDI_IN.31
- net JOYH2: now also J11.3, MIDI_IN.31
Changed lines of the file:
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@@
 </segment>
 </net>
-<net name="B1" class="0">
+<net name="BTN1" class="0">
 <segment>
 <wire x1="121.92" y1="91.44" x2="116.84" y2="91.44" width="0.1524" layer="91"/>
@@
 </segment>
 </net>
-<net name="B2" class="0">
+<net name="BTN2" class="0">
 <segment>
 <wire x1="137.16" y1="91.44" x2="142.24" y2="91.44" width="0.1524" layer="91"/>
@@
 </segment>
 </net>
-<net name="B3" class="0">
+<net name="BTN3" class="0">
 <segment>
 <wire x1="121.92" y1="78.74" x2="116.84" y2="78.74" width="0.1524" layer="91"/>
@@
 </segment>
 </net>
-<net name="B4" class="0">
+<net name="BTN4" class="0">
 <segment>
 <wire x1="137.16" y1="78.74" x2="142.24" y2="78.74" width="0.1524" layer="91"/>
@@
 </segment>
 </net>
-<net name="B5" class="0">
+<net name="BTN5" class="0">
 <segment>
 <label x="119.38" y="66.04" size="1.27" layer="95" rot="R180" xref="yes"/>
@@
 </segment>
 </net>
-<net name="B6" class="0">
+<net name="BTN6" class="0">
 <segment>
 <wire x1="139.7" y1="66.04" x2="144.78" y2="66.04" width="0.1524" layer="91"/>
@@
 </segment>
 </net>
-<net name="B7" class="0">
+<net name="BTN7" class="0">
 <segment>
 <wire x1="121.92" y1="53.34" x2="116.84" y2="53.34" width="0.1524" layer="91"/>
@@
 <net name="JOYH2" class="3">
 <segment>
+<pinref part="J11" gate="G$1" pin="3"/>
+<wire x1="66.04" y1="104.14" x2="73.66" y2="104.14" width="0.1524" layer="91"/>
+<label x="73.66" y="104.14" size="1.016" layer="95" xref="yes"/>
+</segment>
+<segment>
 <wire x1="25.4" y1="190.5" x2="15.24" y2="190.5" width="0.1524" layer="91"/>
 <label x="15.24" y="190.5" size="1.016" layer="95" rot="R180" xref="yes"/>
 <pinref part="TEENSY" gate="G$1" pin="31/A12/PWM/RX4/CS1-0"/>
 </segment>
-</net>
-<net name="JOY_AN_V_M" class="3">
+<segment>
+<pinref part="MIDI_IN" gate="G$1" pin="31"/>
+<wire x1="292.1" y1="88.9" x2="289.56" y2="88.9" width="0.1524" layer="91"/>
+<label x="289.56" y="88.9" size="1.016" layer="95" rot="R180" xref="yes"/>
+</segment>
+</net>
+<net name="JOYV2" class="3">
 <segment>
 <pinref part="J11" gate="G$1" pin="4"/>
@@
 </segment>
 </net>
-<net name="B12" class="0">
+<net name="BTN12" class="0">
 <segment>
 <wire x1="137.16" y1="27.94" x2="142.24" y2="27.94" width="0.1524" layer="91"/>
@@
 </segment>
 </net>
-<net name="B11" class="0">
+<net name="BTN11" class="0">
 <segment>
 <wire x1="121.92" y1="27.94" x2="116.84" y2="27.94" width="0.1524" layer="91"/>
@@
 </segment>
 </net>
-<net name="B10" class="0">
+<net name="BTN10" class="0">
 <segment>
 <wire x1="137.16" y1="40.64" x2="142.24" y2="40.64" width="0.1524" layer="91"/>
@@
 </segment>
 </net>
-<net name="B9" class="0">
+<net name="BTN9" class="0">
 <segment>
 <wire x1="121.92" y1="40.64" x2="116.84" y2="40.64" width="0.1524" layer="91"/>
@@
 </segment>
 </net>
-<net name="B8" class="0">
+<net name="BTN8" class="0">
 <segment>
 <wire x1="137.16" y1="53.34" x2="142.24" y2="53.34" width="0.1524" layer="91"/>
@@
 </segment>
 </net>
-<net name="B13" class="0">
+<net name="BTN13" class="0">
 <segment>
 <pinref part="S5" gate="G$1" pin="1"/>
@@
 </segment>
 </net>
-<net name="B14" class="0">
+<net name="BTN14" class="0">
 <segment>
 <pinref part="S6" gate="G$1" pin="1"/>
@@
 </segment>
 </net>
-<net name="B15" class="0">
+<net name="BTN15" class="0">
 <segment>
 <pinref part="S7" gate="G$1" pin="1"/>
@@
 </segment>
 </net>
-<net name="JOY_AN_V_S" class="3">
+<net name="JOYV1" class="3">
 <segment>
 <pinref part="J10" gate="G$1" pin="4"/>
@@
 </segment>
 </net>
-<net name="JOY_AN_H_S" class="3">
+<net name="JOYH1" class="3">
 <segment>
 <pinref part="J10" gate="G$1" pin="3"/>
@@
 </segment>
 </net>
-<net name="JOY_BTN_S" class="0">
+<net name="JOYB1" class="0">
 <segment>
 <pinref part="J10" gate="G$1" pin="5"/>
@@
 </segment>
 </net>
-<net name="JOY_BTN_M" class="0">
+<net name="JOYB2" class="0">
 <segment>
 <pinref part="J11" gate="G$1" pin="5"/>
@@
 </segment>
 </net>
-<net name="B16" class="0">
+<net name="BTN16" class="0">
 <segment>
 <pinref part="S8" gate="G$1" pin="1"/>
@@
 </segment>
 </net>
-<net name="JOY_AN_H_M" class="3">
-<segment>
-<pinref part="J11" gate="G$1" pin="3"/>
-<wire x1="66.04" y1="104.14" x2="73.66" y2="104.14" width="0.1524" layer="91"/>
-<label x="73.66" y="104.14" size="1.016" layer="95" xref="yes"/>
-</segment>
-<segment>
-<pinref part="MIDI_IN" gate="G$1" pin="31"/>
-<wire x1="292.1" y1="88.9" x2="289.56" y2="88.9" width="0.1524" layer="91"/>
-<label x="289.56" y="88.9" size="1.016" layer="95" rot="R180" xref="yes"/>
-</segment>
-</net>
