File: PCBs/MOL/MOL-v2-2.brd (EAGLE design)
At the start: 138.8 x 49.3 mm, 32 parts, among them J1 SERVO1, J10 JOY1, J11 JOY2, J2 SERVO2, J4 ACTUATORS, J5 POWER-5V, J6 AN5, J7 AN6, J8 AN7, J9 AN8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

Commit message: python done
Connections:
- net M_AIN renamed M_INA
- net M_BIN renamed M_INB
Changed lines of the file:
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@@
 <contactref element="TEENSY" pad="36"/>
 </signal>
-<signal name="M_AIN">
+<signal name="M_INA">
 <contactref element="J4" pad="2"/>
 <contactref element="TEENSY" pad="45"/>
-</signal>
-<signal name="M_BIN">
-<contactref element="J4" pad="4"/>
-<contactref element="TEENSY" pad="46"/>
 </signal>
 <signal name="JOYH2" class="3">
@@
 <contactref element="RN2" pad="8"/>
 </signal>
+<signal name="M_INB">
+<contactref element="J4" pad="4"/>
+<contactref element="TEENSY" pad="46"/>
+<wire x1="42.754" y1="27.23" x2="108.827" y2="32.377" width="0" layer="19" extent="1-1"/>
+</signal>
 </signals>
