File: PCBs/MOL/MOL-v2-2.sch (EAGLE design)
At the start: 34 parts, among them J1 SERVO1, J10 JOY1, J11 JOY2, J2 SERVO2, J4 ACTUATORS, J5 POWER-5V, J6 AN5, J7 AN6, J8 AN7, J9 AN8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

Commit message: python done
Connections:
- net M_AIN renamed M_INA
- net M_BIN renamed M_INB
- removed net N$3: MIDI_OUT.0
- removed net N$4: MIDI_OUT.1
- removed net N$5: MIDI_OUT.2
- removed net N$6: MIDI_OUT.3
- removed net N$7: MIDI_OUT.4
- removed net N$8: MIDI_OUT.5
- net LED1: now also MIDI_OUT.0
- net LED2: now also MIDI_OUT.1
- net LED3: now also MIDI_OUT.2
- net LED4: now also MIDI_OUT.3
- net LED5: now also MIDI_OUT.4
- net LED6: now also MIDI_OUT.5
