File: PCBs/MOD/MOD-v2-2.sch (EAGLE design)
At the start: 40 parts, among them J1 SERVO1, J10 JOY1, J11 JOY2, J12 RPi-Reset, J2 SERVO2, J3 RPi, J4 ACTUATORS, J5 Battery, J6 AN5, J7 AN6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

Commit message: attiny added to MOD pcb
Parts:
- added C1: 10uF, resistor:C-USC0805
- J12: value RPi-Reset -> RPi-Shutdown
- J6, J7, J8, J9: device SparkFun-Connectors:M031X03_NO_SILK -> SparkFun-Connectors:M03LOCK
- R1: device resistor:R-US_0204/7 -> rcl:R-US_M0805
- R2: value 2.2k -> 2.2K; device resistor:R-US_0204/7 -> rcl:R-US_M0805
- R3: value 3.3k -> 3.3K; device resistor:R-US_0204/7 -> rcl:R-US_M0805
- U1: value ATTINY85SU -> ATTINY85
Connections:
- net +5V: now also R1.1; no longer R1.2
- net +5V-BATTERY: now also C1.1
- net GND: now also C1.2, R3.2; no longer R3.1
- net N$2: now also R1.2; no longer R1.1
- net N$5: now also R2.2, R3.1; no longer R2.1, R3.2
- net PI-REST: now also R2.1; no longer R2.2
Other:
- moved on the sheet: J12, J5, R1, R2, R3, SW2
