File: PCBs/MOD/MOD-v2-3a.brd (EAGLE design)
At the start: 100 x 100 mm, 46 parts, among them J12 RPi-Shutdown, J17 +5V (Main), J3 TO Pi, J4 ACTUATORS, J5 +5V (Pi), SW2 500SSP1S2M2QEA, U1 ATTINY85, U2 A2982

Commit message: DRC on MOD pcb v2-3a
Parts:
- moved C1 3.16 mm to (48.0, 18.0)
- moved R1 3.16 mm to (39.0, 18.0)
- moved R2 3.16 mm to (42.0, 18.0)
- moved R3 3.16 mm to (45.0, 18.0)
- moved U2 2.24 mm to (59.3, 78.0)
- moved J3 1.79 mm to (26.1, 102.0)
- moved J17 1.06 mm to (59.3, 102.0)
- moved J5 1.02 mm to (85.6, 102.0)
- moved TEENSY 0.51 mm to (52.0, 99.9)
Routing:
- net GND: track 487.2 -> 552.0 mm, vias 5 -> 4
- net +3V3: track 456.2 -> 515.7 mm, vias 3 -> 6
- net +5V: track 204.7 -> 258.6 mm, vias 5 -> 11
- net N$2: track 171.5 -> 117.9 mm
- net PWM_4: track 68.3 -> 45.3 mm
- net PWM_15: track 77.9 -> 99.1 mm, vias 2 -> 6
- net PWM_16: track 44.8 -> 64.9 mm
- net AGND: track 421.7 -> 402.3 mm
- net PWM14: track 39.4 -> 58.6 mm
- net AN5: track 96.0 -> 115.2 mm, vias 3 -> 4
- net PWM_7: track 43.3 -> 25.7 mm, vias 1 -> 0
- net B4: track 59.2 -> 43.0 mm, vias 3 -> 0
- net PWM_2: track 73.3 -> 89.2 mm, vias 1 -> 2
- net PWM_1: track 94.6 -> 110.4 mm, vias 2 -> 5
- net PWM_3: track 48.2 -> 63.1 mm, vias 1 -> 3
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
Commit message: DRC on MOD pcb v2-3a
Parts:
- added J1: Teensy-5V, SparkFun-Connectors:1X02_LOCK
- C1: device resistor:C0805 -> resistor:C050-024X044
- R1, R2, R3: device rcl:M0805 -> rcl:0204/7
- U1: device attiny85:ATTINY85 -> CMU-ArtFab:DIL08
- moved LED1 19.0 mm to (44.0, 69.0)
- moved U1 4.56 mm to (61.7, 40.8), turned to 270 degrees
- moved STRIP3 3.61 mm to (81.0, 51.0), flipped to the bottom
- moved RELAY1 3.00 mm to (72.2, 73.5)
- moved STRIP2 3.00 mm to (81.0, 38.0), flipped to the bottom
- moved STRIP4 3.00 mm to (81.0, 64.1)
- moved U$2 2.24 mm to (25.8, 36.2)
- moved J17 1.00 mm to (60.3, 102.0)
- moved U2 1.00 mm to (60.3, 78.0)
- flipped J4 to the bottom
- flipped STRIP1 to the bottom
- flipped STRIP5 to the bottom
- flipped STRIP6 to the bottom
Connections:
- new net N$7: J1.1, TEENSY.VIN
- net +5V: now also J1.2; no longer TEENSY.VIN
Routing:
- net GND: track 552.0 -> 459.6 mm, vias 4 -> 7
- net AN1: track 138.3 -> 195.4 mm, vias 3 -> 2
- net B3: track 40.6 -> 84.1 mm, vias 0 -> 2
- net AN10: track 114.5 -> 154.7 mm, vias 7 -> 6
- net +3V3: track 515.7 -> 555.3 mm, vias 6 -> 7
- net N$2: track 117.9 -> 82.2 mm, vias 0 -> 2
- net AGND: track 402.3 -> 436.7 mm, vias 4 -> 5
- net PWM15: track 74.2 -> 43.1 mm, vias 3 -> 2
- net AN9: track 126.1 -> 155.8 mm, vias 9 -> 8
- net AN6: track 95.3 -> 124.9 mm, vias 4 -> 2
- net N$7: track 0.00 -> 28.3 mm
- net AN4: track 117.6 -> 93.5 mm
- net B1: track 65.4 -> 87.2 mm, vias 1 -> 2
- net PWM_16: track 64.9 -> 44.2 mm, vias 2 -> 3
- net N$5: track 116.3 -> 95.9 mm
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