File: PCBs/MOD/MOD-v2-3a.sch (EAGLE design)
At the start: 48 parts, among them J12 RPi-Shutdown, J17 +5V (Main), J3 TO Pi, J4 ACTUATORS, J5 +5V (Pi), SW2 500SSP1S2M2QEA, U1 ATTINY85, U2 A2982

Commit message: DRC on MOD pcb v2-3a
Parts:
- added J1: Teensy-5V, SparkFun-Connectors:CONN_02LOCK
- C1: device resistor:C-USC0805 -> resistor:C-US050-024X044
- R1, R2, R3: device rcl:R-US_M0805 -> rcl:R-US_0204/7
- U1: device attiny85:ATTINY85SU -> CMU-ArtFab:ATTINY85
Connections:
- new net N$7: J1.1, TEENSY.VIN
- net +5V: now also J1.2; no longer TEENSY.VIN
