File: PCBs/MOD/MOD-v2-3c.brd (EAGLE design)
At the start: 100 x 100 mm, 47 parts, among them J1 Teensy-5V, J12 RPi-Shutdown, J17 +5V (Main), J3 TO Pi, J4 ACTUATORS, J5 +5V (Pi), SW2 500SSP1S2M2QEA, U1 ATTINY85, U2 A2982

Commit message: all thru-hole parts, design checked by Jake and Daniel, re-routed with 24mil traces for power
Routing:
- net GND: track 0.00 -> 470.6 mm, vias 0 -> 15
- net B11: track 182.1 -> 37.7 mm, vias 11 -> 2
- net B9: track 149.5 -> 35.4 mm, vias 9 -> 1
- net N$6: track 0.00 -> 75.4 mm, vias 0 -> 3
- net +5V: track 297.3 -> 239.5 mm, vias 9 -> 6
- net AN9: track 152.8 -> 206.5 mm, vias 12 -> 7
- net PWM1: track 63.8 -> 12.1 mm, vias 2 -> 0
- net AGND: track 375.4 -> 414.3 mm, vias 1 -> 8
- net PWM_2: track 107.1 -> 68.7 mm, vias 5 -> 2
- net PWM13: track 60.8 -> 23.6 mm, vias 4 -> 2
- net AN3: track 83.1 -> 119.0 mm
- net PWM2: track 44.9 -> 10.8 mm, vias 3 -> 0
- net AN5: track 87.4 -> 120.6 mm, vias 0 -> 2
- net AN10: track 137.2 -> 167.7 mm
- net B8: track 70.3 -> 40.9 mm, vias 6 -> 1
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- removed copper zone on layer 16, net GND
- removed copper zone on layer 1, net N$6
