File: PCBs/MOD/MOD-v2-4.sch (EAGLE design)
At the start: 49 parts, among them J1 Teensy-5V, J12 RPi-Shutdown, J17 +5V IN (Main), J3 +5V OUT (to Pi), J4 ACTUATORS, J5 +5V IN (Pi), SW2 500SSP1S2M2QEA, U1 ATTINY85, U2 A2982

Commit message: new MOD teensy board
Connections:
- net GND: now also U$2.NC1
Changed lines of the file:
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@@
 <wire x1="177.8" y1="22.86" x2="180.34" y2="22.86" width="0.1524" layer="91"/>
 <wire x1="180.34" y1="22.86" x2="180.34" y2="20.32" width="0.1524" layer="91"/>
+<pinref part="U$2" gate="G$1" pin="NC1"/>
+<wire x1="177.8" y1="22.86" x2="177.8" y2="20.32" width="0.1524" layer="91"/>
+<junction x="177.8" y="22.86"/>
 </segment>
 <segment>
