File: PCBs/MOD/MOD-v2-6.brd (EAGLE design)
At the start: 100 x 100 mm, 47 parts, among them J1 Teensy-5V, J12 RPi-Shutdown, J17 +5V IN (Main), J3 +5V OUT (to Pi), J4 ACTUATORS, J5 +5V IN (Pi), SW2 500SSP1S2M2QEA, U1 ATTINY85, U2 A2982

Commit message: new boards
Parts:
- removed S1A1, S3A5, S5A9: AN5, SparkFun-Connectors:1X03_LOCK
- removed S1A2, S3A6, S5A10: AN6, SparkFun-Connectors:1X03_LOCK
- removed S2A3, S4A7, S6A11: AN7, SparkFun-Connectors:1X03_LOCK
- removed S2A4, S4A8, S6A12: AN8, SparkFun-Connectors:1X03_LOCK
- added S1-A1, S3-A5, S5-A9: AN5, SparkFun-Connectors:1X03_LOCK
- added S1-A2, S3-A6, S5-A10: AN6, SparkFun-Connectors:1X03_LOCK
- added S2-A3, S4-A7, S6-A11: AN7, SparkFun-Connectors:1X03_LOCK
- added S2-A4, S4-A8, S6-A12: AN8, SparkFun-Connectors:1X03_LOCK
- moved R2 165.7 mm to (175.9, 112.4), turned to 270 degrees
- moved R3 151.2 mm to (172.3, 112.4), turned to 90 degrees
- moved KNOB3 150.6 mm to (146.1, 95.4)
- moved KNOB4 146.9 mm to (160.6, 95.2)
- moved SW2 141.1 mm to (151.2, 114.7)
- moved STRIP5 140.9 mm to (155.3, 32.7)
- moved U$2 140.6 mm to (157.3, 65.2)
- moved STRIP6 139.0 mm to (155.1, 5.80)
- moved C1 122.5 mm to (142.7, 116.7)
- moved S2 118.0 mm to (131.6, 80.2)
- moved S4 115.6 mm to (159.3, 79.4)
- moved U2 112.5 mm to (172.3, 65.1)
- moved LED1 110.6 mm to (139.2, 137.1)
- moved U1 105.2 mm to (132.1, 116.0)
- moved R1 102.5 mm to (139.4, 127.4), turned to 90 degrees
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Connections:
- net N$6 renamed RELAY-PWR
- net +3V3: now also S1-A1.1, S1-A2.1, S2-A3.1, S2-A4.1, S3-A5.1, S3-A6.1, S4-A7.1, S4-A8.1, S5-A10.1, S5-A9.1, S6-A11.1, S6-A12.1; no longer S1A1.1, S1A2.1, S2A3.1, S2A4.1, S3A5.1, S3A6.1, S4A7.1, S4A8.1, S5A10.1, S5A9.1, S6A11.1, S6A12.1
- net AGND: now also S1-A1.2, S1-A2.2, S2-A3.2, S2-A4.2, S3-A5.2, S3-A6.2, S4-A7.2, S4-A8.2, S5-A10.2, S5-A9.2, S6-A11.2, S6-A12.2; no longer S1A1.2, S1A2.2, S2A3.2, S2A4.2, S3A5.2, S3A6.2, S4A7.2, S4A8.2, S5A10.2, S5A9.2, S6A11.2, S6A12.2
- net AN1: now also S1-A1.3; no longer S1A1.3
- net AN10: now also S5-A10.3; no longer S5A10.3
- net AN11: now also S6-A11.3; no longer S6A11.3
- net AN12: now also S6-A12.3; no longer S6A12.3
- net AN2: now also S1-A2.3; no longer S1A2.3
- net AN3: now also S2-A3.3; no longer S2A3.3
- net AN4: now also S2-A4.3; no longer S2A4.3
- net AN5: now also S3-A5.3; no longer S3A5.3
- net AN6: now also S3-A6.3; no longer S3A6.3
- net AN7: now also S4-A7.3; no longer S4A7.3
- net AN8: now also S4-A8.3; no longer S4A8.3
- net AN9: now also S5-A9.3; no longer S5A9.3
- net PWM_1: now also U2.13; no longer U2.20
- net PWM_10: now also U$2.14; no longer U$2.19
- net PWM_11: now also U$2.15; no longer U$2.18
- net PWM_12: now also U$2.16; no longer U$2.17
- net PWM_13: now also U$2.17; no longer U$2.16
- net PWM_14: now also U$2.18; no longer U$2.15
- net PWM_15: now also U$2.19; no longer U$2.14
- net PWM_16: now also U$2.20; no longer U$2.13
- net PWM_2: now also U2.14; no longer U2.19
- net PWM_3: now also U2.15; no longer U2.18
- net PWM_4: now also U2.16; no longer U2.17
- net PWM_5: now also U2.17; no longer U2.16
- net PWM_6: now also U2.18; no longer U2.15
- net PWM_7: now also U2.19; no longer U2.14
- net PWM_8: now also U2.20; no longer U2.13
- net PWM_9: now also U$2.13; no longer U$2.20
Other:
- board text added: "+5V IN (Main)"
- board text added: "+5V IN (pi)"
- board text added: "+5V OUT (to Pi)"
