File: PCBs/MOD/MOD-v2-5.sch (EAGLE design)
At the start: 49 parts, among them J1 Teensy-5V, J12 RPi-Shutdown, J17 +5V IN (Main), J3 +5V OUT (to Pi), J4 ACTUATORS, J5 +5V IN (Pi), SW2 500SSP1S2M2QEA, U1 ATTINY85, U2 A2982

Commit message: MOD-v2-5 routed
Parts:
- added R4, R5, R6, R7: 330, rcl:R-US_0204/7
- renumbered S1-A1 to S1-AN1, S1-A2 to S1-AN2, S2-A3 to S2-AN3, S2-A4 to S2-AN4, S3-A5 to S3-AN5, S3-A6 to S3-AN6, S4-A7 to S4-AN7, S4-A8 to S4-AN8
Connections:
- new net N$3: R4.2, S1.A
- new net N$4: R5.2, S2.A
- new net N$6: R6.2, S3.A
- new net N$8: R7.2, S4.A
- net PWM_13: now also R4.1; no longer S1.A
- net PWM_14: now also R5.1; no longer S2.A
- net PWM_15: now also R6.1; no longer S3.A
- net PWM_16: now also R7.1; no longer S4.A
Other:
- moved on the sheet: S1, S2, S3, S4, U$2, U2
